File: Starling WiPSU Ver_0.1/Starling WiPSU ver_0.1.kicad_pcb (KiCad board)
At the start: 2 copper layers, 50 x 19 mm, 25 parts, among them CON1 9V/2A, P1 CONN_01X01, P2 ESP8266 - 01, P3 CONN_01X01, P4 CONN_01X01, P5 CONN_01X01, P6 2.3" Display Conn, P7 0.8" Display Conn, Q1 MOSFET_N, Q2 MOSFET_N, Q3 BC847, SW1 SW_PUSH, U1 L78S05, U2 1117-3.3

Commit message: Wifi and PSU ver0.1 updated
Parts:
- removed the C2 at (115.5, 91.0)
- removed the CON1 at (93.5, 89.0)
- removed the P1 at (91.5, 80.5)
- removed the P4 at (43.5, 135.5)
- removed P5: CONN_01X01, EE:M3_mounting
- removed the P6 at (110.6, 78.8)
- removed P7: 0.8" Display Conn, connect:1.27mm_smd_Header
- removed the Q1 at (108.5, 87.0)
- removed the Q2 at (105.0, 93.5)
- removed the Q3 at (138.5, 79.5)
- removed the SW1 at (111.0, 83.0)
- removed the U1 at (112.5, 90.0)
- added C1: 0.1uF, Capacitors_SMD:C_0603, F.Cu at (164.5, 94.5)
- added C1: 0.1uF, Capacitors_SMD:C_0603, F.Cu at (164.5, 114.0)
- added C1: 0.1uF, Capacitors_SMD:C_0603, F.Cu at (104.5, 114.0)
- added C2: CP1, Capacitors_Tantalum_SMD:TantalC_SizeA_EIA-3216_Wave, F.Cu at (158.5, 82.5)
- added C2: CP1, Capacitors_Tantalum_SMD:TantalC_SizeA_EIA-3216_Wave, F.Cu at (158.5, 102.0)
- added C2: CP1, Capacitors_Tantalum_SMD:TantalC_SizeA_EIA-3216_Wave, F.Cu at (98.5, 102.0)
- added C2: CP1, Capacitors_Tantalum_SMD:TantalC_SizeA_EIA-3216_Wave, F.Cu at (98.5, 82.5)
- added C3: 4u7, Capacitors_Tantalum_SMD:TantalC_SizeA_EIA-3216_Wave, F.Cu at (158.5, 79.5)
- added C3: 4u7, Capacitors_Tantalum_SMD:TantalC_SizeA_EIA-3216_Wave, F.Cu at (158.5, 99.0)
- added C3: 4u7, Capacitors_Tantalum_SMD:TantalC_SizeA_EIA-3216_Wave, F.Cu at (98.5, 99.0)
- added C4: 10u, Capacitors_Tantalum_SMD:TantalC_SizeA_EIA-3216_Wave, F.Cu at (169.5, 82.0)
- added C4: 10u, Capacitors_Tantalum_SMD:TantalC_SizeA_EIA-3216_Wave, F.Cu at (169.5, 101.5)
- added C4: 10u, Capacitors_Tantalum_SMD:TantalC_SizeA_EIA-3216_Wave, F.Cu at (109.5, 101.5)
- added C5: 0.1u, Capacitors_SMD:C_0603, B.Cu at (152.2, 92.5)
- added C5: 0.1u, Capacitors_SMD:C_0603, B.Cu at (152.2, 112.0)
- added C5: 0.1u, Capacitors_SMD:C_0603, B.Cu at (92.2, 112.0)
- added C6: 2u2, Capacitors_SMD:C_0603, B.Cu at (172.6, 92.2)
- added C6: 2u2, Capacitors_SMD:C_0603, B.Cu at (172.6, 111.8)
- added C6: 2u2, Capacitors_SMD:C_0603, B.Cu at (112.6, 111.8)
- added CON1: 9V/2A, Connect:BARREL_JACK, F.Cu at (154.1, 88.9)
- added CON1: 9V/2A, Connect:BARREL_JACK, F.Cu at (154.1, 108.5)
- added CON1: 9V/2A, Connect:BARREL_JACK, F.Cu at (94.0, 108.5)
- added CON1: 9V/2A, Connect:BARREL_JACK, F.Cu at (94.0, 88.9)
- added G***: LOGO, Logo:Logo_silk_OSHW_6x6mm, B.Cu at (194.2, 79.5)
- added G***: LOGO, Logo:Logo_silk_OSHW_6x6mm, B.Cu at (194.2, 99.0)
- added G***: LOGO, Logo:Logo_silk_OSHW_6x6mm, B.Cu at (134.2, 99.0)
- added G***: LOGO, Logo:Logo_silk_OSHW_6x6mm, B.Cu at (134.2, 79.5)
- added P1: HC-05 Bluetooth, Pin_Headers:Pin_Header_Straight_1x06, B.Cu at (188.8, 81.5)
- added P1: HC-05 Bluetooth, Pin_Headers:Pin_Header_Straight_1x06, B.Cu at (188.8, 101.0)
- added P1: HC-05 Bluetooth, Pin_Headers:Pin_Header_Straight_1x06, B.Cu at (128.8, 101.0)
- added P1: HC-05 Bluetooth, Pin_Headers:Pin_Header_Straight_1x06, B.Cu at (128.8, 81.5)
- added P2: ESP8266 - 01, ESP8266:ESP-01, B.Cu at (185.0, 85.0)
- added P2: ESP8266 - 01, ESP8266:ESP-01, B.Cu at (185.0, 104.5)
- added P2: ESP8266 - 01, ESP8266:ESP-01, B.Cu at (125.0, 104.5)
- added P3: CONN_01X01, EE:M3_mounting, F.Cu at (202.0, 80.5)
- added P3: CONN_01X01, EE:M3_mounting, F.Cu at (202.0, 100.0)
- added P3: CONN_01X01, EE:M3_mounting, F.Cu at (142.0, 100.0)
- added P4: CONN_01X01, EE:M3_mounting, F.Cu at (149.8, 80.8)
- added P4: CONN_01X01, EE:M3_mounting, F.Cu at (149.8, 100.3)
- added P4: CONN_01X01, EE:M3_mounting, F.Cu at (89.8, 100.3)
- added P4: CONN_01X01, EE:M3_mounting, F.Cu at (89.8, 80.8)
- added P6: 2.3" Display Conn, Pin_Headers:Pin_Header_Straight_1x06, F.Cu at (165.6, 79.1)
- added P6: 2.3" Display Conn, Pin_Headers:Pin_Header_Straight_1x06, F.Cu at (165.6, 98.6)
- added P6: 2.3" Display Conn, Pin_Headers:Pin_Header_Straight_1x06, F.Cu at (105.6, 98.6)
- added P6: 2.3" Display Conn, Pin_Headers:Pin_Header_Straight_1x06, F.Cu at (105.6, 79.1)
- added Q1: BSS138, SMD Ttorransis:sot23, B.Cu at (178.8, 91.4)
- added Q1: BSS138, SMD Ttorransis:sot23, B.Cu at (178.8, 111.0)
- added Q1: BSS138, SMD Ttorransis:sot23, B.Cu at (118.8, 111.0)
- added Q1: BSS138, SMD Ttorransis:sot23, B.Cu at (118.8, 91.4)
- added Q2: BSS138, SMD Ttorransis:sot23, B.Cu at (175.1, 90.2)
- added Q2: BSS138, SMD Ttorransis:sot23, B.Cu at (175.1, 109.8)
- added Q2: BSS138, SMD Ttorransis:sot23, B.Cu at (115.1, 109.8)
- added Q2: BSS138, SMD Ttorransis:sot23, B.Cu at (115.1, 90.2)
- added Q3: BC847, TO_SOT_Packages_SMD:SOT-23, F.Cu at (184.0, 79.5)
- added Q3: BC847, TO_SOT_Packages_SMD:SOT-23, F.Cu at (184.0, 99.0)
- added Q3: BC847, TO_SOT_Packages_SMD:SOT-23, F.Cu at (124.0, 99.0)
- added Q3: BC847, TO_SOT_Packages_SMD:SOT-23, F.Cu at (124.0, 79.5)
- added R1: 470K, Resistors_SMD:R_0603, B.Cu at (178.9, 94.4)
- added R1: 470K, Resistors_SMD:R_0603, B.Cu at (178.9, 114.0)
- added R1: 470K, Resistors_SMD:R_0603, B.Cu at (119.0, 114.0)
- added R2: 100K, Resistors_SMD:R_0603, B.Cu at (176.2, 93.9)
- added R2: 100K, Resistors_SMD:R_0603, B.Cu at (176.2, 113.4)
- added R2: 100K, Resistors_SMD:R_0603, B.Cu at (116.2, 113.4)
- added R3: 47K, Resistors_SMD:R_0603, B.Cu at (178.4, 86.8)
- added R3: 47K, Resistors_SMD:R_0603, B.Cu at (178.4, 106.3)
- added R3: 47K, Resistors_SMD:R_0603, B.Cu at (118.4, 106.3)
- added R4: 330E, Resistors_SMD:R_0603, F.Cu at (181.2, 81.2)
- added R4: 330E, Resistors_SMD:R_0603, F.Cu at (181.2, 100.8)
- added R4: 330E, Resistors_SMD:R_0603, F.Cu at (121.2, 100.8)
- added R5: R, Resistors_SMD:R_0603, F.Cu at (166.5, 84.5)
- added R5: R, Resistors_SMD:R_0603, F.Cu at (166.5, 104.0)
- added R5: R, Resistors_SMD:R_0603, F.Cu at (106.5, 104.0)
- added R5: R, Resistors_SMD:R_0603, F.Cu at (106.5, 84.5)
- added R6: R, Resistors_SMD:R_0603, F.Cu at (165.1, 82.7)
- added R6: R, Resistors_SMD:R_0603, F.Cu at (165.1, 102.2)
- added R6: R, Resistors_SMD:R_0603, F.Cu at (105.0, 102.2)
- added R6: R, Resistors_SMD:R_0603, F.Cu at (105.0, 82.7)
- added SP1: SPEAKER, Buzzers_Beepers:Buzzer_12x9.5RM7.6, B.Cu at (199.5, 90.0)
- added SP1: SPEAKER, Buzzers_Beepers:Buzzer_12x9.5RM7.6, B.Cu at (199.5, 109.5)
- added SP1: SPEAKER, Buzzers_Beepers:Buzzer_12x9.5RM7.6, B.Cu at (139.5, 109.5)
- added SW1: SW_PUSH, sw:smd_push, B.Cu at (148.5, 89.0)
- added SW1: SW_PUSH, sw:smd_push, B.Cu at (148.5, 108.5)
- added SW1: SW_PUSH, sw:smd_push, B.Cu at (88.5, 108.5)
- added SW1: SW_PUSH, sw:smd_push, B.Cu at (88.5, 89.0)
- added U1: LM317S, TO_SOT_Packages_SMD:TO-263-3Lead, F.Cu at (165.8, 89.5)
- added U1: LM317S, TO_SOT_Packages_SMD:TO-263-3Lead, F.Cu at (165.8, 109.0)
- added U1: LM317S, TO_SOT_Packages_SMD:TO-263-3Lead, F.Cu at (105.8, 109.0)
- added U1: LM317S, TO_SOT_Packages_SMD:TO-263-3Lead, F.Cu at (105.8, 89.5)
- added U2: 1117-3.3, TO_SOT_Packages_SMD:SOT-223, F.Cu at (194.0, 87.5)
- added U2: 1117-3.3, TO_SOT_Packages_SMD:SOT-223, F.Cu at (194.0, 107.0)
- added U2: 1117-3.3, TO_SOT_Packages_SMD:SOT-223, F.Cu at (134.0, 107.0)
- C1: value 0.33uF -> 0.1uF
- C5, C6, R1, R2, R3: moved to B.Cu
- moved SP1 39.8 mm to (139.5, 90.0), turned to 90 degrees
- moved C3 21.1 mm to (98.5, 79.5)
- moved C5 21.0 mm to (92.2, 92.5), turned to 0 degrees
- moved R3 16.8 mm to (118.4, 86.8), turned to 0 degrees
- moved C4 16.2 mm to (109.5, 82.0)
- moved P2 16.0 mm to (125.0, 85.0)
- moved R1 13.8 mm to (119.0, 94.4), turned to 180 degrees
- moved R4 13.3 mm to (121.2, 81.2), turned to 270 degrees
- moved U2 13.2 mm to (134.0, 87.5), turned to 0 degrees
- moved R2 13.0 mm to (116.2, 93.9), turned to 270 degrees
- moved P3 12.5 mm to (142.0, 80.5)
- moved C6 10.7 mm to (112.6, 92.2), turned to 90 degrees
- moved C1 5.41 mm to (104.5, 94.5), turned to 180 degrees
Routing:
- net GND: track 0.00 -> 479.1 mm, vias 0 -> 12
- net +5V: track 0.00 -> 330.0 mm, vias 0 -> 4
- net +3V3: track 0.00 -> 324.2 mm, vias 0 -> 12
- net /RESET: track 0.00 -> 183.9 mm
- net /RX: track 0.00 -> 158.5 mm
- net /TX: track 0.00 -> 85.1 mm
- net Net-(Q3-Pad3): track 0.00 -> 80.5 mm
- net Net-(C1-Pad1): track 0.00 -> 44.2 mm
- net /GPIO0: track 0.00 -> 37.5 mm
- net /BUZ: track 0.00 -> 31.7 mm
- net Net-(P2-Pad3): track 0.00 -> 28.8 mm
- net Net-(C6-Pad1): track 0.00 -> 22.4 mm
- net Net-(R5-Pad1): track 0.00 -> 17.2 mm
- net Net-(Q1-PadD): track 0.00 -> 16.8 mm
- net Net-(Q3-Pad1): track 0.00 -> 7.20 mm
Other:
- board size 50 x 19 mm -> 120 x 39 mm
- net class Default: trace_width 0.25 -> 0.35; via_dia 0.6 -> 0.8
- board text added: "Comp"
- board text added: "ExploreEmbedded.com"
- board text added: "Sold"
