File: Starling WiPSU Ver_0.1/Starling WiPSU ver_0.1.sch (KiCad schematic (older format))
At the start: 23 parts, among them CON1 9V/2A, P2 ESP8266 - 01, P3 CONN_01X01, P4 CONN_01X01, P6 2.3\" Display Conn, P7 0.8\" Display Conn, Q1 MOSFET_N, Q2 MOSFET_N, Q3 BC847, SW1 SW_PUSH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

Commit message: Wifi and PSU ver0.1 updated
Parts:
- removed C2: 0.1uF, Capacitors_SMD:C_0603, symbol C
- removed P7: 0.8\" Display Conn, connect:1.27mm_smd_Header, symbol CONN_01X07
- removed U1: L78S05, TO_SOT_Packages_THT:TO-220_Neutral123_Horizontal_MountedFromLS_LargePads, symbol LM7805CT
- added C2: CP1, Capacitors_Tantalum_SMD:TantalC_SizeA_EIA-3216_Wave, symbol CP1
- added P1: HC-05 Bluetooth, Pin_Headers:Pin_Header_Straight_1x06, symbol CONN_01X06
- added R5, R6: R, Resistors_SMD:R_0603, symbol R
- added U1: LM317S, TO_SOT_Packages_SMD:TO-263-3Lead, symbol LM317S
- C1: value 0.33uF -> 0.1uF
- Q1, Q2: value MOSFET_N -> BSS138
Connections:
- net +5V: now also C2.1, P1.5 (P5), R6.1, U1.2 (OUT)
- net GND: now also C2.2, P1.4 (P4), R5.2
- net RX: now also P1.3 (P3)
- net TX: now also P1.2 (P2)
- net at C1.1, CON1.1: now also U1.3 (IN)
- new net: R5.1, R6.2, U1.1 (ADJ)
